File: MobileCloud(PCB)/MobileCloud.kicad_pcb (KiCad board)
At the start: 2 copper layers, 49 parts, among them J1 , J10 , J11 , J12 , J2 , J3 , J4 , J5 , J6 , J7 , J8 , J9 , U1 L298HN, U2 RPM5.0-6.0, U3 RPM5.0-6.0, U4 L298HN, U5 LD1117S33TR_SOT223, U6 ATmega328P-PU, Y1 16MHz Crystal

Commit message: Add files via upload
Parts:
- added J13: , Connector_PinSocket_2.00mm:PinSocket_1x02_P2.00mm_Vertical, F.Cu at (90.2, 75.6)
- moved J12 54.0 mm to (73.7, 59.1), turned to 270 degrees
- moved C6 42.6 mm to (77.5, 44.5), turned to 0 degrees
- moved J9 39.2 mm to (77.5, 17.4), turned to 90 degrees
- moved C8 36.8 mm to (85.7, 75.6), turned to 270 degrees
- moved Y1 36.4 mm to (81.3, 49.5), turned to 0 degrees
- moved J7 35.0 mm to (60.3, 34.9), turned to 180 degrees
- moved FB3 34.9 mm to (61.6, 39.4), turned to 270 degrees
- moved C4 34.3 mm to (64.8, 38.1), turned to 0 degrees
- moved R2 33.9 mm to (88.9, 54.6), turned to 180 degrees
- moved J11 31.9 mm to (87.6, 59.1), turned to 270 degrees
- moved U5 30.2 mm to (55.2, 26.6)
- moved J10 24.1 mm to (94.0, 59.1), turned to 270 degrees
- moved C7 23.5 mm to (90.2, 44.5), turned to 180 degrees
- moved R1 22.5 mm to (99.1, 55.2)
- moved J1 21.3 mm to (55.9, 41.3), turned to 180 degrees
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Connections:
- U6 pad 14: Net-(U4-Pad10) -> Net-(U1-Pad12)
- U6 pad 15: Net-(U1-Pad11) -> Net-(U1-Pad10)
- U6 pad 16: Net-(U4-Pad11) -> Net-(U1-Pad11)
- U6 pad 17: Net-(U1-Pad10) -> Net-(U4-Pad10)
- U6 pad 18: Net-(U1-Pad12) -> Net-(U4-Pad12)
- U6 pad 19: Net-(U4-Pad12) -> Net-(U4-Pad11)
Routing:
- net Net-(C4-Pad1): track 41.6 -> 111.8 mm
- net Net-(U1-Pad12): track 120.9 -> 52.2 mm
- net Net-(U1-Pad11): track 84.3 -> 40.4 mm
- net Net-(U1-Pad10): track 77.2 -> 40.4 mm
- net Net-(C6-Pad2): track 44.1 -> 21.3 mm, vias 2 -> 0
- net Net-(U4-Pad10): track 24.2 -> 44.6 mm
- net Net-(D1-Pad2): track 13.5 -> 31.2 mm
- net Net-(C7-Pad2): track 43.8 -> 26.2 mm, vias 2 -> 0
- net Net-(C5-Pad1): track 19.0 -> 33.6 mm
- net Net-(J13-Pad2): track 0.00 -> 13.2 mm
- net Net-(C2-Pad1): track 39.5 -> 28.6 mm
- net Net-(U4-Pad12): track 50.9 -> 41.0 mm
- net Net-(J13-Pad1): track 0.00 -> 9.15 mm
- net Net-(C3-Pad1): track 126.8 -> 120.2 mm
- net GNDREF: track 0.00 -> 6.08 mm
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Other:
- rule trace_min: 0.2 -> 0.508

Commit message: Add files via upload
Parts:
- removed REF**: AssmannHeatsink, MobileCloud(PCB):V7466x_AssManHeatsink
- added D17: LED, LED_THT:LED_D3.0mm, F.Cu at (87.6, 83.8)
- added D18: LED, LED_THT:LED_D3.0mm, F.Cu at (63.5, 27.3)
- added D19: LED, LED_THT:LED_D3.0mm, F.Cu at (50.2, 19.7)
- added HS1: Assmann_Heatsink_V7466, MobileCloud(PCB):V7466x_AssManHeatsink, F.Cu at (74.9, 102.9)
- added R3: 330, Resistor_THT:R_Axial_DIN0207_L6.3mm_D2.5mm_P10.16mm_Horizontal, F.Cu at (64.1, 77.5)
- added R4: 330, Resistor_THT:R_Axial_DIN0207_L6.3mm_D2.5mm_P10.16mm_Horizontal, F.Cu at (66.7, 21.6)
- added R5: 120, Resistor_THT:R_Axial_DIN0207_L6.3mm_D2.5mm_P10.16mm_Horizontal, F.Cu at (49.5, 24.1)
- moved J1 5.72 mm to (50.2, 41.3), turned to 0 degrees
- moved C5 4.62 mm to (60.3, 19.1), turned to 180 degrees
- moved J6 3.17 mm to (71.8, 27.3)
- moved C8 3.16 mm to (82.6, 74.9), turned to 0 degrees
- moved D10 0.64 mm to (94.7, 117.3)
- moved D13 0.64 mm to (98.6, 104.6)
- moved D14 0.64 mm to (98.6, 117.3)
- moved D9 0.64 mm to (94.7, 104.6)
- moved J13 0.63 mm to (90.2, 74.9)
- moved J4 0.63 mm to (90.8, 114.9)
- moved J9 0.23 mm to (77.5, 17.1)
Connections:
- J1 pad 1: GNDREF -> Net-(C1-Pad1)
- J1 pad 2: Net-(C1-Pad1) -> GNDREF
- U2 pad C1: Net-(U2-PadC1) -> Net-(C2-Pad1)
- U3 pad C1: Net-(U3-PadC1) -> Net-(C2-Pad1)
Routing:
- net Net-(C3-Pad1): track 120.2 -> 144.6 mm
- net Net-(D17-Pad2): track 0.00 -> 14.5 mm
- net Net-(C2-Pad1): track 28.6 -> 40.4 mm
- net Net-(C5-Pad1): track 33.6 -> 43.9 mm
- net Net-(D18-Pad1): track 0.00 -> 6.58 mm
- net Net-(D19-Pad1): track 0.00 -> 4.71 mm
- net Net-(C4-Pad1): track 111.8 -> 115.2 mm
- net Net-(J6-Pad2): track 17.2 -> 14.1 mm
- net Net-(J6-Pad1): track 20.8 -> 17.6 mm
- net Net-(FB2-Pad2): track 8.52 -> 10.8 mm
- net Net-(FB3-Pad2): track 6.61 -> 8.90 mm
- net Net-(C8-Pad1): track 6.92 -> 5.00 mm
- net Net-(J13-Pad2): track 13.2 -> 12.3 mm
- net Net-(D10-Pad1): track 18.2 -> 19.0 mm
- net Net-(D13-Pad2): track 29.3 -> 29.9 mm
- added copper zone on B.Cu, net GNDREF
- added copper zone on F.Cu, net GNDREF
Other:
- board outline added: 58.4 x 118.1 mm
- board text added: "REV C"
- board text added: "SDSU SENIOR DESIGN"
- board text added: "SMILE CLOUD9"
- board text added: "Tx Rx"
